File: PCB_Hardware/Boards/DBCAN/DBCAN_V1.0/DBCAN_V1.0.kicad_sch (KiCad schematic)
At the start: 2 parts

Commit message: First version of DBCAN board
Other:
- removed sheet EEPROM
- sheet MCU ports: added none; removed EEPROM_SCL, EEPROM_SDA
- moved on the sheet: H1, H2
