File: PCB_Hardware/Boards/DBCAN/DBCAN_V1.0/MCU.kicad_sch (KiCad schematic)
At the start: 9 parts, among them J1 Conn_ARM_SWD_TagConnect_TC203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, U1 STM32G0B1KBT6TR, Y1 ASEMB-8.000MHZ-XY-T

Commit message: First version of DBCAN board
Parts:
- removed C7: 100n, Capacitor_SMD:C_0402_1005Metric, symbol Device:C
- removed C8: 10n, Capacitor_SMD:C_0402_1005Metric, symbol Device:C
- removed D7: BLUE, LED_SMD:LED_0603_1608Metric, symbol Device:LED
- removed J1: Conn_ARM_SWD_TagConnect_TC2030-NL, Connector:Tag-Connect_TC2030-IDC-NL_2x03_P1.27mm_Vertical, symbol Connector:Conn_ARM_SWD_TagConnect_TC2030-NL
- removed R53: 2.2k, Resistor_SMD:R_0402_1005Metric, symbol Device:R
- added C3, C4, C5: 100n, Capacitor_SMD:C_0402_1005Metric, symbol Device:C
- added D8: BLUE, LED_SMD:LED_0603_1608Metric, symbol Device:LED
- added J1: Conn_ARM_SWD_TagConnect_TC2030, Connector:Tag-Connect_TC2030-IDC-FP_2x03_P1.27mm_Vertical, symbol Connector:Conn_ARM_SWD_TagConnect_TC2030
- added R17: 2.2k, Resistor_SMD:R_0402_1005Metric, symbol Device:R
- added R18: 0, Resistor_SMD:R_0402_1005Metric, symbol Device:R
- added TP14, TP4, TP5: TestPoint, TestPoint:TestPoint_Pad_D1.0mm, symbol Connector:TestPoint
- C1: Cost (none) -> 0.001; Manufacturer_Name (none) -> Samsung Electro-Mechanics; Manufacturer_Part_Number (none) -> CL10A475KO8NNNC; Source (none) -> LCSC
- C2: Cost (none) -> 0.0011; Manufacturer_Name (none) -> YAGEO; Manufacturer_Part_Number (none) -> CC0402KRX7R7BB104; Source (none) -> LCSC
- U1: value STM32G0B1KBT6TR -> STM32G0B1KBT6; Cost (none) -> 3.80; Manufacturer_Name (none) -> ST Microelectronics; Manufacturer_Part_Number (none) -> STM32G0B1KBT6; Source (none) -> LCSC
- Y1: value ASEMB-8.000MHZ-XY-T -> ASEM1-24.000MHZ-LC-T; Cost (none) -> 2.77; Manufacturer_Name (none) -> Abracon LLC; Manufacturer_Part_Number (none) -> ASEM1-24.000MHZ-LC-T; Source (none) -> Digikey
Connections:
- net +3.3V: now also C3.1, C4.1, J1.1 (VCC)
- net CANFD_RX1: now also U1.29 (PB5); no longer U1.32 (PB8)
- net CANFD_RX2: now also U1.32 (PB8); no longer U1.15 (PB0)
- net CANFD_TX1: now also U1.30 (PB6); no longer U1.1 (PB9)
- net CANFD_TX2: now also U1.1 (PB9); no longer U1.16 (PB1)
- net GND: now also C3.2, C4.2, C5.1, J1.5 (GND), R17.1
- net NRST: now also C5.2, J1.3 (~{RESET}), TP14.1
- net SEQ1: now also U1.3 (PC15); no longer U1.31 (PB7)
- net SEQ2: now also U1.7 (PA0); no longer U1.17 (PB2)
- net SWCLK: now also J1.4 (SWCLK), TP4.1
- net SWDIO: now also J1.2 (SWDIO), TP5.1
- net TERM_R1: now also U1.31 (PB7); no longer U1.30 (PB6)
- net TERM_R2: now also U1.26 (PA15); no longer U1.18 (PA8)
- net at U1.2 (PC14): now also R18.1; no longer Y1.3 (OUT)
- net EEPROM_SCL: no longer names the net of U1.27 (PB3)
- net EEPROM_SDA: no longer names the net of U1.28 (PB4)
- new net: D8.1 (K), R17.2
- new net: D8.2 (A), U1.18 (PA8)
- new net: R18.2, Y1.3 (OUT)
- no-connect marks 14 -> 16
Other:
- moved on the sheet: C1, C2, U1
