File: PCB_Hardware/Boards/DBCAN/DBCAN_V1.0/USB.kicad_sch (KiCad schematic)
At the start: 17 parts, among them J11 GT-USB-7010ASV, U10 TPD2E2U06DCK, U3 MCP1802T-3302I/OT

Commit message: Completed board layout and tweaks to schematic. Added 3D model lib
Parts:
- added TP1, TP2, TP3: TestPoint, TestPoint:TestPoint_Pad_D1.0mm, symbol Connector:TestPoint
Connections:
- net +3.3V: now also TP2.1
- net +5V: now also TP1.1
- net GND: now also TP3.1

Commit message: First version of DBCAN board
Parts:
- added TP12, TP13: TestPoint, TestPoint:TestPoint_Pad_D1.0mm, symbol Connector:TestPoint
- C11: renamed from C37; Cost (none) -> 0.001; Manufacturer_Name (none) -> Samsung Electro-Mechanics; Manufacturer_Part_Number (none) -> CL10A475KO8NNNC; Source (none) -> LCSC
- C12: renamed from C38; Cost (none) -> 0.0011; Manufacturer_Name (none) -> YAGEO; Manufacturer_Part_Number (none) -> CC0402KRX7R7BB104; Source (none) -> LCSC
- C13: renamed from C39; Cost (none) -> 0.0064; Manufacturer_Name (none) -> Samsung Electro-Mechanics; Manufacturer_Part_Number (none) -> CL10B105KA8NNNC; Source (none) -> LCSC
- C14: renamed from C40; Cost (none) -> 0.0064; Manufacturer_Name (none) -> Samsung Electro-Mechanics; Manufacturer_Part_Number (none) -> CL10B105KA8NNNC; Source (none) -> LCSC
- D1: renamed from D4; Cost (none) -> 0.01; Manufacturer_Name (none) -> XINGLIGHT; Manufacturer_Part_Number (none) -> XL-1608VRC-06; Source (none) -> LCSC
- D2: renamed from D10; Cost (none) -> 0.12; Manufacturer_Name (none) -> Littelfuse; Manufacturer_Part_Number (none) -> SMAJ5.0A; Source (none) -> LCSC
- D3: renamed from D1; Cost (none) -> 0.01; Manufacturer_Name (none) -> XINGLIGHT; Manufacturer_Part_Number (none) -> XL-1608VRC-06; Source (none) -> LCSC
- F1: value MF-PSMF050X-2 -> BSMD0805-050-24V; Cost (none) -> 0.06; Manufacturer_Part_Number (none) -> BSMD0805-050-24V; Source (none) -> LCSC
- J2: renamed from J11; Cost (none) -> 0.09; Manufacturer_Name (none) -> G-Switch; Manufacturer_Part_Number (none) -> GT-USB-7010ASV; Source (none) -> LCSC
- R3: renamed from R50; Cost (none) -> 0.0004; Manufacturer_Name (none) -> YAGEO; Manufacturer_Part_Number (none) -> RC0402FR-075M9L; Source (none) -> LCSC
- R4: renamed from R49; Cost (none) -> 0.0004; Manufacturer_Name (none) -> YAGEO; Manufacturer_Part_Number (none) -> RC0402FR-075M9L; Source (none) -> LCSC
- R5: renamed from R47; Cost (none) -> 0.0007; Manufacturer_Name (none) -> YAGEO; Manufacturer_Part_Number (none) -> RC0402JR-075K1L; Source (none) -> LCSC
- R6: renamed from R48; Cost (none) -> 0.0007; Manufacturer_Name (none) -> YAGEO; Manufacturer_Part_Number (none) -> RC0402JR-075K1L; Source (none) -> LCSC
- R7: renamed from R51; value 22 -> 0; Cost (none) -> 0.0007; Manufacturer_Name (none) -> YAGEO; Manufacturer_Part_Number (none) -> RC0402JR-070RL; Source (none) -> LCSC
- R8: renamed from R52; value 22 -> 0; Cost (none) -> 0.0007; Manufacturer_Name (none) -> YAGEO; Manufacturer_Part_Number (none) -> RC0402JR-070RL; Source (none) -> LCSC
- U2: renamed from U3; Cost (none) -> 0.72; Manufacturer_Name (none) -> Microchip Technology; Manufacturer_Part_Number (none) -> MCP1802T-3302I/OT; Source (none) -> Digikey
- U3: renamed from U10; Cost (none) -> 0.16; Manufacturer_Name (none) -> Texas Instruments; Manufacturer_Part_Number (none) -> TPD2E2U06DCKR; Source (none) -> LCSC
- renumbered TP2 to TP1, TP1 to TP2
Connections:
- net D+: now also TP13.1
- net D-: now also TP12.1
Other:
- moved on the sheet: TP3
