File: PCB_Hardware/Boards/DBCAN/DBCAN_V1.0/CANFD.kicad_sch (KiCad schematic)
At the start: 23 parts, among them J2 SM04B-PASS-TBT, J3 SM04B-PASS-TBT, Q1 SI2302, Q2 SI2302, Q3 SI2302, Q4 SI2302, U2 TCAN1048AVDMTRQ1

Commit message: First version of DBCAN board
Parts:
- added TP10, TP11, TP6, TP7, TP8, TP9: TestPoint, TestPoint:TestPoint_Pad_D1.0mm, symbol Connector:TestPoint
- C15: renamed from C3; Cost (none) -> 0.0011; Manufacturer_Name (none) -> YAGEO; Manufacturer_Part_Number (none) -> CC0402KRX7R7BB104; Source (none) -> LCSC
- C16: renamed from C6; Cost (none) -> 0.0011; Manufacturer_Name (none) -> YAGEO; Manufacturer_Part_Number (none) -> CC0402KRX7R7BB104; Source (none) -> LCSC
- C17: renamed from C4; Cost (none) -> 0.0012; Manufacturer_Name (none) -> YAGEO; Manufacturer_Part_Number (none) -> CC0402KRX7R9BB472; Source (none) -> LCSC
- C18: renamed from C5; Cost (none) -> 0.0012; Manufacturer_Name (none) -> YAGEO; Manufacturer_Part_Number (none) -> CC0402KRX7R9BB472; Source (none) -> LCSC
- D4: renamed from D6; Cost (none) -> 0.02; Manufacturer_Name (none) -> UMW; Manufacturer_Part_Number (none) -> PESD5V0L1UL; Source (none) -> LCSC
- D5: renamed from D2; Cost (none) -> 0.09; Manufacturer_Name (none) -> Nexperia; Manufacturer_Part_Number (none) -> PESD1CAN; Source (none) -> LCSC
- D6: renamed from D3; Cost (none) -> 0.09; Manufacturer_Name (none) -> Nexperia; Manufacturer_Part_Number (none) -> PESD1CAN; Source (none) -> LCSC
- D7: renamed from D5; Cost (none) -> 0.02; Manufacturer_Name (none) -> UMW; Manufacturer_Part_Number (none) -> PESD5V0L1UL; Source (none) -> LCSC
- J3: renamed from J2; Cost (none) -> 0.58; Manufacturer_Name (none) -> JST; Manufacturer_Part_Number (none) -> SM04B-PASS-TBT; Source (none) -> LCSC
- J4: renamed from J3; Cost (none) -> 0.58; Manufacturer_Name (none) -> JST; Manufacturer_Part_Number (none) -> SM04B-PASS-TBT; Source (none) -> LCSC
- Q1, Q2, Q3, Q4: Manufacturer_Name (none) -> VISHAY; Manufacturer_Part_Number (none) -> Si2302CDS-T1-GE3; Source (none) -> LCSC
- R10: renamed from R2; value 60 -> 60.4; Cost (none) -> 0.0026; Manufacturer_Name (none) -> YAGEO; Manufacturer_Part_Number (none) -> RC0805FR-0760R4L; Source (none) -> LCSC
- R11: renamed from R3; value 60 -> 60.4; Cost (none) -> 0.0026; Manufacturer_Name (none) -> YAGEO; Manufacturer_Part_Number (none) -> RC0805FR-0760R4L; Source (none) -> LCSC
- R12: renamed from R4; value 60 -> 60.4; Cost (none) -> 0.0026; Manufacturer_Name (none) -> YAGEO; Manufacturer_Part_Number (none) -> RC0805FR-0760R4L; Source (none) -> LCSC
- R13: renamed from R5; Cost (none) -> 0.0007; Manufacturer_Name (none) -> YAGEO; Manufacturer_Part_Number (none) -> RC0402JR-1310KL; Source (none) -> LCSC
- R14: renamed from R6; Cost (none) -> 0.0007; Manufacturer_Name (none) -> YAGEO; Manufacturer_Part_Number (none) -> RC0402JR-1310KL; Source (none) -> LCSC
- R15: renamed from R7; value 100k -> 1k; Cost (none) -> 0.0009; Manufacturer_Name (none) -> YAGEO; Manufacturer_Part_Number (none) -> AC0402JR-071KL; Source (none) -> LCSC
- R16: renamed from R8; value 100k -> 1k; Cost (none) -> 0.0009; Manufacturer_Name (none) -> YAGEO; Manufacturer_Part_Number (none) -> AC0402JR-071KL; Source (none) -> LCSC
- R9: renamed from R1; value 60 -> 60.4; Cost (none) -> 0.0026; Manufacturer_Name (none) -> YAGEO; Manufacturer_Part_Number (none) -> RC0805FR-0760R4L; Source (none) -> LCSC
- U4: renamed from U2; Cost (none) -> 2.51; Source (none) -> Digikey
Connections:
- net CANFD1+: now also TP6.1
- net CANFD1-: now also TP7.1
- net CANFD2+: now also TP9.1
- net CANFD2-: now also TP10.1
- net SEQ1_PIN: now reaches D4.1 (K), J3.3 (Pin_3), R15.1
- net SEQ1_PIN: now also TP8.1
- net SEQ2_PIN: now reaches D7.1 (K), J4.3 (Pin_3), R16.1
- net SEQ2_PIN: now also TP11.1
Other:
- moved on the sheet: D4

Commit message: Created organization around the symbol lib and did a first pass layout of the BDLC
Parts:
- U4: symbol DBRobot:TCAN1048AVDMTRQ1 -> DBRobot_CAN_Transceiver:TCAN1048AVDMTRQ1
Changed lines of the file:
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@@
 	)
 	(symbol
-		(lib_id "DBRobot:TCAN1048AVDMTRQ1")
+		(lib_id "DBRobot_CAN_Transceiver:TCAN1048AVDMTRQ1")
 		(at 60.96 78.74 0)
 		(unit 1)
