File: PCB_Hardware/Boards/BLDC/BLDC_V1.0/OR_Inputs.kicad_sch (KiCad schematic)
At the start: 9 parts, among them U12 LM66100DCK, U13 LM66100DCK

Commit message: Add DBcan transport refactor, BLDC V1.0 schematic + sim work, HAL submodule
- DBcan: replace bare-register driver with vendor-agnostic transport abstraction (core/, transports/, refactored bootloader driver, README)
- Add stm32g4xx_hal_driver as Firmware/libs submodule
- Add HAL config for BLDC board (stm32g4xx_hal_conf.h)
- BLDC V1.0: schematic edits across 10 sheets (footprint assignments, repositioning); design-doc README (gate-driver constraints, FET selection / TPH3R70APL, thermal analysis)
- ngspice simulation workflow (cap sweeps, half-bridge slow turn-on)
- Ignore .obsidian/ vault state and large simulation CSV exports
Parts:
- C39: footprint (none) -> Capacitor_SMD:C_0402_1005Metric
- D11: footprint (none) -> LED_SMD:LED_0603_1608Metric
- R49, R52, R53, R54: footprint (none) -> Resistor_SMD:R_0402_1005Metric
Changed lines of the file:
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@@
 			)
 		)
-		(property "Footprint" ""
+		(property "Footprint" "LED_SMD:LED_0603_1608Metric"
 			(at 176.53 57.15 0)
 			(hide yes)
@@
 			)
 		)
-		(property "Footprint" ""
+		(property "Footprint" "Resistor_SMD:R_0402_1005Metric"
 			(at 111.76 94.488 90)
 			(hide yes)
@@
 			)
 		)
-		(property "Footprint" ""
+		(property "Footprint" "Capacitor_SMD:C_0402_1005Metric"
 			(at 158.4452 66.04 0)
 			(hide yes)
@@
 			)
 		)
-		(property "Footprint" ""
+		(property "Footprint" "Resistor_SMD:R_0402_1005Metric"
 			(at 103.632 66.04 90)
 			(hide yes)
@@
 			)
 		)
-		(property "Footprint" ""
+		(property "Footprint" "Resistor_SMD:R_0402_1005Metric"
 			(at 167.132 62.23 90)
 			(hide yes)
@@
 			)
 		)
-		(property "Footprint" ""
+		(property "Footprint" "Resistor_SMD:R_0402_1005Metric"
 			(at 127.762 68.58 90)
 			(hide yes)
