File: PCB_Hardware/Boards/BLDC/BLDC_V1.0/OR_Inputs.kicad_sch (KiCad schematic)
At the start: 9 parts, among them U12 LM66100DCK, U13 LM66100DCK

Commit message: minor BLDC changes and production files for ordering
Parts:
- C39: Manufacturer_Part_Number (none) -> CL05A106MP5NUNC
- D11: Manufacturer_Part_Number (none) -> XINGLIGHT XL-1608SURC-06
- R49, R52, R53, R54: Manufacturer_Part_Number (none) -> CQ02WGJ0104TCE
- R50: value 5k -> 5.1k; Manufacturer_Part_Number (none) -> RC0402JR-075K1L
- U12, U13: Manufacturer_Part_Number (none) -> LM66100DCK
Changed lines of the file:
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@@
+			)
+		)
+		(property "Manufacturer_Part_Number" "XINGLIGHT XL-1608SURC-06"
+			(at 176.53 57.15 0)
+			(hide yes)
+			(show_name no)
+			(do_not_autoplace no)
+			(effects
+				(font
+					(size 1.27 1.27)
+				)
 			)
 		)
@@
 			)
 		)
+		(property "Manufacturer_Part_Number" " CQ02WGJ0104TCE"
+			(at 111.76 92.71 90)
+			(hide yes)
+			(show_name no)
+			(do_not_autoplace no)
+			(effects
+				(font
+					(size 1.27 1.27)
+				)
+			)
+		)
 		(pin "2"
 		)
@@
 			)
 		)
+		(property "Manufacturer_Part_Number" " CL05A106MP5NUNC"
+			(at 157.48 62.23 0)
+			(hide yes)
+			(show_name no)
+			(do_not_autoplace no)
+			(effects
+				(font
+					(size 1.27 1.27)
+				)
+			)
+		)
 		(pin "2"
 		)
@@
 			)
 		)
-		(property "Value" "5k"
+		(property "Value" "5.1k"
 			(at 186.69 63.4999 0)
 			(show_name no)
@@
 		)
 		(property "Description" "Resistor"
+			(at 184.15 62.23 0)
+			(hide yes)
+			(show_name no)
+			(do_not_autoplace no)
+			(effects
+				(font
+					(size 1.27 1.27)
+				)
+			)
+		)
+		(property "Manufacturer_Part_Number" "RC0402JR-075K1L"
 			(at 184.15 62.23 0)
 			(hide yes)
@@
 			)
 		)
+		(property "Manufacturer_Part_Number" " CQ02WGJ0104TCE"
+			(at 105.41 66.04 0)
+			(hide yes)
+			(show_name no)
+			(do_not_autoplace no)
+			(effects
+				(font
+					(size 1.27 1.27)
+				)
+			)
+		)
 		(pin "2"
 		)
@@
 			)
 		)
+		(property "Manufacturer_Part_Number" "LM66100DCK"
+			(at 139.7 90.17 0)
+			(hide yes)
+			(show_name no)
+			(do_not_autoplace no)
+			(effects
+				(font
+					(size 1.27 1.27)
+				)
+			)
+		)
 		(pin "1"
 		)
@@
 			)
 		)
+		(property "Manufacturer_Part_Number" "LM66100DCK"
+			(at 139.7 59.69 0)
+			(hide yes)
+			(show_name no)
+			(do_not_autoplace no)
+			(effects
+				(font
+					(size 1.27 1.27)
+				)
+			)
+		)
 		(pin "1"
 		)
@@
 			)
 		)
+		(property "Manufacturer_Part_Number" " CQ02WGJ0104TCE"
+			(at 168.91 62.23 0)
+			(hide yes)
+			(show_name no)
+			(do_not_autoplace no)
+			(effects
+				(font
+					(size 1.27 1.27)
+				)
+			)
+		)
 		(pin "2"
 		)
@@
 			(at 129.54 68.58 0)
 			(hide yes)
+			(show_name no)
+			(do_not_autoplace no)
+			(effects
+				(font
+					(size 1.27 1.27)
+				)
+			)
+		)
+		(property "Manufacturer_Part_Number" " CQ02WGJ0104TCE"
+			(at 129.54 68.58 0)
+			(hide yes)
