File: PCB_Hardware/Boards/BLDC/BLDC_V1.0/BLDC_V1.0.kicad_sch (KiCad schematic)
At the start: 0 parts

Commit message: Created organization around the symbol lib and did a first pass layout of the BDLC
Parts:
- added H1, H2, H3, H4: MountingHole, MountingHole:MountingHole_3.2mm_M3, symbol Mechanical:MountingHole
