File: PCB_Hardware/Boards/BLDC/BLDC_V1.0/Break.kicad_sch (KiCad schematic)
At the start: 7 parts, among them J5 Conn_01x02_Socket, Q10 BC847, Q9 TPH3R70APL

Commit message: Add DBcan transport refactor, BLDC V1.0 schematic + sim work, HAL submodule
- DBcan: replace bare-register driver with vendor-agnostic transport abstraction (core/, transports/, refactored bootloader driver, README)
- Add stm32g4xx_hal_driver as Firmware/libs submodule
- Add HAL config for BLDC board (stm32g4xx_hal_conf.h)
- BLDC V1.0: schematic edits across 10 sheets (footprint assignments, repositioning); design-doc README (gate-driver constraints, FET selection / TPH3R70APL, thermal analysis)
- ngspice simulation workflow (cap sweeps, half-bridge slow turn-on)
- Ignore .obsidian/ vault state and large simulation CSV exports
Parts:
- D5: footprint (none) -> Diode_SMD:D_SOD-123F
- J5: footprint (none) -> Connector_JST:JST_XH_S2B-XH-A-1_1x02_P2.50mm_Horizontal
- R18, R19, R20: footprint (none) -> Resistor_SMD:R_0402_1005Metric
Changed lines of the file:
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@@
 			)
 		)
-		(property "Footprint" ""
+		(property "Footprint" "Diode_SMD:D_SOD-123F"
 			(at 161.29 87.63 0)
 			(hide yes)
@@
 			)
 		)
-		(property "Footprint" ""
+		(property "Footprint" "Resistor_SMD:R_0402_1005Metric"
 			(at 148.59 100.838 90)
 			(hide yes)
@@
 			)
 		)
-		(property "Footprint" ""
+		(property "Footprint" "Connector_JST:JST_XH_S2B-XH-A-1_1x02_P2.50mm_Horizontal"
 			(at 181.61 86.36 0)
 			(hide yes)
@@
 			)
 		)
-		(property "Footprint" ""
+		(property "Footprint" "Resistor_SMD:R_0402_1005Metric"
 			(at 124.46 107.188 90)
 			(hide yes)
@@
 			)
 		)
-		(property "Footprint" ""
+		(property "Footprint" "Resistor_SMD:R_0402_1005Metric"
 			(at 135.382 93.98 90)
 			(hide yes)

Commit message: Created organization around the symbol lib and did a first pass layout of the BDLC
Parts:
- Q9: footprint (none) -> DBRobot:SOP AdvanceN_TOS
Changed lines of the file:
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@@
 			)
 		)
-		(property "Footprint" ""
+		(property "Footprint" "DBRobot:SOP AdvanceN_TOS"
 			(at 163.83 96.52 0)
 			(hide yes)
