File: PCB_Hardware/Boards/BLDC/BLDC_V1.0/Break.kicad_sch (KiCad schematic)
At the start: 7 parts, among them J5 Conn_01x02_Socket, Q10 BC847, Q9 TPH3R70APL

Commit message: minor BLDC changes and production files for ordering
Parts:
- D5: Manufacturer_Part_Number (none) -> SS10150
- Q9: Manufacturer_Part_Number (none) -> TPH3R70APL
- R18: Manufacturer_Part_Number (none) -> HP02WAJ0103TCE
- R19: Manufacturer_Part_Number (none) -> 0402WGJ047JTCE
- R20: Manufacturer_Part_Number (none) -> CQ02WGJ0102TCE
Changed lines of the file:
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@@
+			)
+		)
+		(property "Manufacturer_Part_Number" "SS10150"
+			(at 161.29 87.63 90)
+			(hide yes)
+			(show_name no)
+			(do_not_autoplace no)
+			(effects
+				(font
+					(size 1.27 1.27)
+				)
 			)
 		)
@@
 			)
 		)
+		(property "Manufacturer_Part_Number" "0402WGJ047JTCE"
+			(at 148.59 99.06 90)
+			(hide yes)
+			(show_name no)
+			(do_not_autoplace no)
+			(effects
+				(font
+					(size 1.27 1.27)
+				)
+			)
+		)
 		(pin "2"
 		)
@@
 			)
 		)
+		(property "Manufacturer_Part_Number" "TPH3R70APL"
+			(at 158.75 99.06 0)
+			(hide yes)
+			(show_name no)
+			(do_not_autoplace no)
+			(effects
+				(font
+					(size 1.27 1.27)
+				)
+			)
+		)
 		(pin "4"
 		)
@@
 			)
 		)
+		(property "Manufacturer_Part_Number" "CQ02WGJ0102TCE"
+			(at 124.46 105.41 90)
+			(hide yes)
+			(show_name no)
+			(do_not_autoplace no)
+			(effects
+				(font
+					(size 1.27 1.27)
+				)
+			)
+		)
 		(pin "2"
 		)
@@
 			(at 137.16 93.98 0)
 			(hide yes)
+			(show_name no)
+			(do_not_autoplace no)
+			(effects
+				(font
+					(size 1.27 1.27)
+				)
+			)
+		)
+		(property "Manufacturer_Part_Number" " HP02WAJ0103TCE"
+			(at 137.16 93.98 0)
+			(hide yes)
