File: PCB_Hardware/Boards/BLDC/BLDC_V1.0/Fan.kicad_sch (KiCad schematic)
At the start: 12 parts, among them J14 47053-1000, Q11 BSS138

Commit message: Created organization around the symbol lib and did a first pass layout of the BDLC
Parts:
- R58: value 0 -> 10k
Changed lines of the file:
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@@
 			)
 		)
-		(property "Value" "0"
+		(property "Value" "10k"
 			(at 124.46 96.5199 0)
 			(show_name no)
