File: PCB_Hardware/Boards/BLDC/BLDC_V1.0/Fan.kicad_sch (KiCad schematic)
At the start: 12 parts, among them J14 47053-1000, Q11 BSS138

Commit message: minor BLDC changes and production files for ordering
Parts:
- C57: Manufacturer_Part_Number (none) -> CC0402ZRY5V6BB104; Price (none) -> 0.0015
- F6: Manufacturer_Part_Number (none) -> MF-PSMF050X-2
- R56: Manufacturer_Part_Number (none) -> RC0402JR-13100RL
- R57: Manufacturer_Part_Number (none) -> CQ02WGJ0104TCE
- R58, R59: Manufacturer_Part_Number (none) -> HP02WAJ0103TCE
- R60: Manufacturer_Part_Number (none) -> CQ02WGJ0102TCE
Changed lines of the file:
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@@
+			)
+		)
+		(property "Manufacturer_Part_Number" "CC0402ZRY5V6BB104"
+			(at 137.16 105.41 0)
+			(hide yes)
+			(show_name no)
+			(do_not_autoplace no)
+			(effects
+				(font
+					(size 1.27 1.27)
+				)
+			)
+		)
+		(property "Price" "0.0015"
+			(at 137.16 105.41 0)
+			(hide yes)
+			(show_name no)
+			(do_not_autoplace no)
+			(effects
+				(font
+					(size 1.27 1.27)
+				)
 			)
 		)
@@
 			)
 		)
+		(property "Manufacturer_Part_Number" "RC0402JR-13100RL"
+			(at 106.68 106.68 90)
+			(hide yes)
+			(show_name no)
+			(do_not_autoplace no)
+			(effects
+				(font
+					(size 1.27 1.27)
+				)
+			)
+		)
 		(pin "2"
 		)
@@
 			)
 		)
+		(property "Manufacturer_Part_Number" "CQ02WGJ0102TCE"
+			(at 157.48 97.79 90)
+			(hide yes)
+			(show_name no)
+			(do_not_autoplace no)
+			(effects
+				(font
+					(size 1.27 1.27)
+				)
+			)
+		)
 		(pin "2"
 		)
@@
 			)
 		)
+		(property "Manufacturer_Part_Number" " HP02WAJ0103TCE"
+			(at 147.32 92.71 0)
+			(hide yes)
+			(show_name no)
+			(do_not_autoplace no)
+			(effects
+				(font
+					(size 1.27 1.27)
+				)
+			)
+		)
 		(pin "2"
 		)
@@
 			)
 		)
+		(property "Manufacturer_Part_Number" "MF-PSMF050X-2"
+			(at 186.69 87.63 0)
+			(hide yes)
+			(show_name no)
+			(do_not_autoplace no)
+			(effects
+				(font
+					(size 1.27 1.27)
+				)
+			)
+		)
 		(pin "1"
 		)
@@
 		)
 		(property "Description" "Resistor"
+			(at 111.76 113.03 0)
+			(hide yes)
+			(show_name no)
+			(do_not_autoplace no)
+			(effects
+				(font
+					(size 1.27 1.27)
+				)
+			)
+		)
+		(property "Manufacturer_Part_Number" " CQ02WGJ0104TCE"
 			(at 111.76 113.03 0)
 			(hide yes)
@@
 			(at 121.92 95.25 0)
 			(hide yes)
+			(show_name no)
+			(do_not_autoplace no)
+			(effects
+				(font
+					(size 1.27 1.27)
+				)
+			)
+		)
+		(property "Manufacturer_Part_Number" " HP02WAJ0103TCE"
+			(at 121.92 95.25 0)
+			(hide yes)
