File: PCB_Hardware/Boards/BLDC/BLDC_V1.0/Temp_Sense.kicad_sch (KiCad schematic)
At the start: 7 parts, among them J6 Conn_01x02_Socket

Commit message: Add DBcan transport refactor, BLDC V1.0 schematic + sim work, HAL submodule
- DBcan: replace bare-register driver with vendor-agnostic transport abstraction (core/, transports/, refactored bootloader driver, README)
- Add stm32g4xx_hal_driver as Firmware/libs submodule
- Add HAL config for BLDC board (stm32g4xx_hal_conf.h)
- BLDC V1.0: schematic edits across 10 sheets (footprint assignments, repositioning); design-doc README (gate-driver constraints, FET selection / TPH3R70APL, thermal analysis)
- ngspice simulation workflow (cap sweeps, half-bridge slow turn-on)
- Ignore .obsidian/ vault state and large simulation CSV exports
Parts:
- F3: footprint (none) -> Fuse:Fuse_0805_2012Metric
- J6: footprint (none) -> Connector_JST:JST_XH_S2B-XH-A-1_1x02_P2.50mm_Horizontal
- R22, R23: footprint (none) -> Resistor_SMD:R_0402_1005Metric
Changed lines of the file:
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@@
 			)
 		)
-		(property "Footprint" ""
+		(property "Footprint" "Resistor_SMD:R_0402_1005Metric"
 			(at 106.172 106.68 90)
 			(hide yes)
@@
 			)
 		)
-		(property "Footprint" ""
+		(property "Footprint" "Connector_JST:JST_XH_S2B-XH-A-1_1x02_P2.50mm_Horizontal"
 			(at 185.42 96.52 0)
 			(hide yes)
@@
 			)
 		)
-		(property "Footprint" ""
+		(property "Footprint" "Resistor_SMD:R_0402_1005Metric"
 			(at 148.082 104.14 90)
 			(hide yes)
@@
 			)
 		)
-		(property "Footprint" ""
+		(property "Footprint" "Fuse:Fuse_0805_2012Metric"
 			(at 180.34 96.52 0)
 			(hide yes)

Commit message: Created organization around the symbol lib and did a first pass layout of the BDLC
Parts:
- J6: footprint Connector_JST:JST_XH_S2B-XH-A-1_1x02_P2.50mm_Horizontal -> Connector_JST:JST_GH_SM02B-GHS-TB_1x02-1MP_P1.25mm_Horizontal
- TH1: footprint (none) -> Resistor_SMD:R_0603_1608Metric
Changed lines of the file:
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@@
 			)
 		)
-		(property "Footprint" ""
+		(property "Footprint" "Resistor_SMD:R_0603_1608Metric"
 			(at 107.95 95.25 0)
 			(hide yes)
@@
 			)
 		)
-		(property "Footprint" "Connector_JST:JST_XH_S2B-XH-A-1_1x02_P2.50mm_Horizontal"
+		(property "Footprint" "Connector_JST:JST_GH_SM02B-GHS-TB_1x02-1MP_P1.25mm_Horizontal"
 			(at 185.42 96.52 0)
 			(hide yes)
