File: PCB_Hardware/Boards/BLDC/BLDC_V1.0/Temp_Sense.kicad_sch (KiCad schematic)
At the start: 7 parts, among them J6 Conn_01x02_Socket

Commit message: minor BLDC changes and production files for ordering
Parts:
- F3: Manufacturer_Part_Number (none) -> MF-PSMF050X-2
- R22, R23: Manufacturer_Part_Number (none) -> HP02WAJ0103TCE
Changed lines of the file:
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@@
+			)
+		)
+		(property "Manufacturer_Part_Number" " HP02WAJ0103TCE"
+			(at 107.95 106.68 0)
+			(hide yes)
+			(show_name no)
+			(do_not_autoplace no)
+			(effects
+				(font
+					(size 1.27 1.27)
+				)
 			)
 		)
@@
 			)
 		)
+		(property "Manufacturer_Part_Number" " HP02WAJ0103TCE"
+			(at 149.86 104.14 0)
+			(hide yes)
+			(show_name no)
+			(do_not_autoplace no)
+			(effects
+				(font
+					(size 1.27 1.27)
+				)
+			)
+		)
 		(pin "1"
 		)
@@
 			(at 179.07 91.44 0)
 			(hide yes)
+			(show_name no)
+			(do_not_autoplace no)
+			(effects
+				(font
+					(size 1.27 1.27)
+				)
+			)
+		)
+		(property "Manufacturer_Part_Number" "MF-PSMF050X-2"
+			(at 179.07 91.44 0)
+			(hide yes)
