File: PCB_Hardware/Boards/BLDC/BLDC_V1.0/CANFD.kicad_sch (KiCad schematic)
At the start: 17 parts, among them J1 Conn_01x04_Pin, J2 Conn_01x04_Pin, Q1 SI2302, Q14 SI2302, U3 TCAN1044VDR

Commit message: minor BLDC changes and production files for ordering
Parts:
- C2, C3: Manufacturer_Part_Number (none) -> CC0402ZRY5V6BB104; Price (none) -> 0.0015
- C4: Manufacturer_Part_Number (none) -> CC0402JRX7R6BB473; Price (none) -> 0.0034
- J1, J2: Manufacturer_Part_Number (none) -> JST SM04B-PASS-TB(LF)(SN)
- Q1: Manufacturer_Part_Number (none) -> Si2302CDS-T1-GE3
- R1, R2: Manufacturer_Part_Number (none) -> CQ05W8F604JT5E
- R33: Manufacturer_Part_Number (none) -> 0402WGJ0182TCE
- R34: Manufacturer_Part_Number (none) -> RC0402JR-073K3L
- R35: Manufacturer_Part_Number RC0402JR-1310KL -> HP02WAJ0103TCE
- R36: Manufacturer_Part_Number AC0402JR-071KL -> CQ02WGJ0102TCE
- U3: Manufacturer_Part_Number (none) -> TCAN1044VDR
Changed lines of the file:
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@@
 			)
 		)
-		(property "Manufacturer_Part_Number" "RC0402JR-1310KL"
+		(property "Manufacturer_Part_Number" " HP02WAJ0103TCE"
 			(at 184.15 111.76 0)
 			(hide yes)
@@
 			)
 		)
+		(property "Manufacturer_Part_Number" "0402WGJ0182TCE"
+			(at 193.04 91.44 0)
+			(hide yes)
+			(show_name no)
+			(do_not_autoplace no)
+			(effects
+				(font
+					(size 1.27 1.27)
+				)
+			)
+		)
 		(pin "1"
 		)
@@
 			)
 		)
-		(property "Manufacturer_Part_Number" "AC0402JR-071KL"
+		(property "Manufacturer_Part_Number" "CQ02WGJ0102TCE"
 			(at 194.31 123.19 90)
 			(hide yes)
@@
 			)
 		)
+		(property "Manufacturer_Part_Number" "JST SM04B-PASS-TB(LF)(SN)"
+			(at 214.63 120.65 0)
+			(hide yes)
+			(show_name no)
+			(do_not_autoplace no)
+			(effects
+				(font
+					(size 1.27 1.27)
+				)
+			)
+		)
 		(pin "1"
 		)
@@
 			)
 		)
+		(property "Manufacturer_Part_Number" "CQ05W8F604JT5E"
+			(at 134.62 66.04 90)
+			(hide yes)
+			(show_name no)
+			(do_not_autoplace no)
+			(effects
+				(font
+					(size 1.27 1.27)
+				)
+			)
+		)
 		(pin "1"
 		)
@@
 		)
 		(property "Description" "Unpolarized capacitor"
+			(at 87.63 64.77 0)
+			(hide yes)
+			(show_name no)
+			(do_not_autoplace no)
+			(effects
+				(font
+					(size 1.27 1.27)
+				)
+			)
+		)
+		(property "Manufacturer_Part_Number" "CC0402ZRY5V6BB104"
+			(at 87.63 64.77 0)
+			(hide yes)
+			(show_name no)
+			(do_not_autoplace no)
+			(effects
+				(font
+					(size 1.27 1.27)
+				)
+			)
+		)
+		(property "Price" "0.0015"
 			(at 87.63 64.77 0)
 			(hide yes)
@@
 			)
 		)
+		(property "Manufacturer_Part_Number" "JST SM04B-PASS-TB(LF)(SN)"
+			(at 214.63 83.82 0)
+			(hide yes)
+			(show_name no)
+			(do_not_autoplace no)
+			(effects
+				(font
+					(size 1.27 1.27)
+				)
+			)
+		)
 		(pin "1"
 		)
@@
 			)
 		)
+		(property "Manufacturer_Part_Number" "CC0402ZRY5V6BB104"
+			(at 114.3 64.77 0)
+			(hide yes)
+			(show_name no)
+			(do_not_autoplace no)
+			(effects
+				(font
+					(size 1.27 1.27)
+				)
+			)
+		)
+		(property "Price" "0.0015"
+			(at 114.3 64.77 0)
+			(hide yes)
+			(show_name no)
+			(do_not_autoplace no)
+			(effects
+				(font
+					(size 1.27 1.27)
+				)
+			)
+		)
 		(pin "2"
 		)
@@
 			)
 		)
+		(property "Manufacturer_Part_Number" " RC0402JR-073K3L"
+			(at 193.04 101.6 0)
+			(hide yes)
+			(show_name no)
+			(do_not_autoplace no)
+			(effects
+				(font
+					(size 1.27 1.27)
+				)
+			)
+		)
 		(pin "1"
 		)
@@
 			)
 		)
+		(property "Manufacturer_Part_Number" "TCAN1044VDR"
+			(at 91.44 74.93 0)
+			(hide yes)
+			(show_name no)
+			(do_not_autoplace no)
+			(effects
+				(font
+					(size 1.27 1.27)
+				)
+			)
+		)
 		(pin "4"
 		)
@@
 			)
 		)
+		(property "Manufacturer_Part_Number" "CQ05W8F604JT5E"
+			(at 144.78 66.04 90)
+			(hide yes)
+			(show_name no)
+			(do_not_autoplace no)
+			(effects
+				(font
+					(size 1.27 1.27)
+				)
+			)
+		)
 		(pin "1"
 		)
@@
 			)
 		)
+		(property "Manufacturer_Part_Number" "CC0402JRX7R6BB473"
+			(at 139.7 71.12 0)
+			(hide yes)
+			(show_name no)
+			(do_not_autoplace no)
+			(effects
+				(font
+					(size 1.27 1.27)
+				)
+			)
+		)
+		(property "Price" "0.0034"
+			(at 139.7 71.12 0)
+			(hide yes)
+			(show_name no)
+			(do_not_autoplace no)
+			(effects
+				(font
+					(size 1.27 1.27)
+				)
+			)
+		)
 		(pin "2"
 		)
@@
 			(hide yes)
 			(show_name no)
+			(do_not_autoplace no)
+			(effects
+				(font
+					(size 1.27 1.27)
+				)
+			)
+		)
+		(property "Manufacturer_Part_Number" "Si2302CDS-T1-GE3"
+			(at 154.94 63.5 90)
+			(hide yes)
+			(show_name no)
