File: PCB_Hardware/Boards/BLDC/BLDC_V1.0/EEPROM.kicad_sch (KiCad schematic)
At the start: 4 parts, among them U16 CAT24C512C8UTR

Commit message: minor BLDC changes and production files for ordering
Parts:
- C46: Manufacturer_Part_Number (none) -> CC0402ZRY5V6BB104; Price (none) -> 0.0015
- R27, R28: Manufacturer_Part_Number (none) -> CQ02WGF4701TCE
- U16: Manufacturer_Part_Number (none) -> CAT24C512C8UTR
Changed lines of the file:
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@@
+			)
+		)
+		(property "Manufacturer_Part_Number" "CQ02WGF4701TCE"
+			(at 139.7 88.9 0)
+			(hide yes)
+			(show_name no)
+			(do_not_autoplace no)
+			(effects
+				(font
+					(size 1.27 1.27)
+				)
 			)
 		)
@@
 			)
 		)
+		(property "Manufacturer_Part_Number" "CAT24C512C8UTR"
+			(at 161.29 102.87 0)
+			(hide yes)
+			(show_name no)
+			(do_not_autoplace no)
+			(effects
+				(font
+					(size 1.27 1.27)
+				)
+			)
+		)
 		(pin "5"
 		)
@@
 			)
 		)
+		(property "Manufacturer_Part_Number" "CC0402ZRY5V6BB104"
+			(at 151.13 88.9 0)
+			(hide yes)
+			(show_name no)
+			(do_not_autoplace no)
+			(effects
+				(font
+					(size 1.27 1.27)
+				)
+			)
+		)
+		(property "Price" "0.0015"
+			(at 151.13 88.9 0)
+			(hide yes)
+			(show_name no)
+			(do_not_autoplace no)
+			(effects
+				(font
+					(size 1.27 1.27)
+				)
+			)
+		)
 		(pin "2"
 		)
@@
 			(at 129.54 88.9 0)
 			(hide yes)
+			(show_name no)
+			(do_not_autoplace no)
+			(effects
+				(font
+					(size 1.27 1.27)
+				)
+			)
+		)
+		(property "Manufacturer_Part_Number" "CQ02WGF4701TCE"
+			(at 129.54 88.9 0)
+			(hide yes)
