File: PCB_Hardware/Boards/BLDC/BLDC_V1.0/Encoder.kicad_sch (KiCad schematic)
At the start: 3 parts, among them U2 MT6835GT-STD

Commit message: minor BLDC changes and production files for ordering
Parts:
- C1: Manufacturer_Part_Number (none) -> CC0402ZRY5V6BB104; Price (none) -> 0.0015
- D1: Manufacturer_Part_Number (none) -> SD05T1G
- U2: Manufacturer_Part_Number (none) -> MT6835GT-STD
Changed lines of the file:
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@@
+			)
+		)
+		(property "Manufacturer_Part_Number" "SD05T1G"
+			(at 119.38 72.39 90)
+			(hide yes)
+			(show_name no)
+			(do_not_autoplace no)
+			(effects
+				(font
+					(size 1.27 1.27)
+				)
 			)
 		)
@@
 			)
 		)
+		(property "Manufacturer_Part_Number" "CC0402ZRY5V6BB104"
+			(at 134.62 72.39 0)
+			(hide yes)
+			(show_name no)
+			(do_not_autoplace no)
+			(effects
+				(font
+					(size 1.27 1.27)
+				)
+			)
+		)
+		(property "Price" "0.0015"
+			(at 134.62 72.39 0)
+			(hide yes)
+			(show_name no)
+			(do_not_autoplace no)
+			(effects
+				(font
+					(size 1.27 1.27)
+				)
+			)
+		)
 		(pin "2"
 		)
@@
 			(at 132.08 82.55 0)
 			(hide yes)
+			(show_name no)
+			(do_not_autoplace no)
+			(effects
+				(font
+					(size 1.27 1.27)
+				)
+			)
+		)
+		(property "Manufacturer_Part_Number" "MT6835GT-STD"
+			(at 132.08 82.55 0)
+			(hide yes)
