File: PCB_Hardware/Boards/BLDC/BLDC_V1.0/GPIO.kicad_sch (KiCad schematic)
At the start: 16 parts, among them J8 Conn_02x06_Odd_Even, J9 Conn_01x06_Socket, Q12 BSS84, U14 SRV05-4, U15 TS5A3159ADBVR, U8 SRV05-4, U9 SRV05-4

Commit message: minor BLDC changes and production files for ordering
Parts:
- F1, F2, F4, F5: Manufacturer_Part_Number (none) -> MF-PSMF050X-2
- R25, R26: Manufacturer_Part_Number (none) -> CQ02WGF4701TCE
- U14, U8, U9: Manufacturer_Part_Number (none) -> SRV05-4
- U15: Manufacturer_Part_Number (none) -> TS5A3159ADBVR
Changed lines of the file:
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@@
+			)
+		)
+		(property "Manufacturer_Part_Number" "TS5A3159ADBVR"
+			(at 208.28 123.19 0)
+			(hide yes)
+			(show_name no)
+			(do_not_autoplace no)
+			(effects
+				(font
+					(size 1.27 1.27)
+				)
 			)
 		)
@@
 			)
 		)
+		(property "Manufacturer_Part_Number" "CQ02WGF4701TCE"
+			(at 68.58 49.53 0)
+			(hide yes)
+			(show_name no)
+			(do_not_autoplace no)
+			(effects
+				(font
+					(size 1.27 1.27)
+				)
+			)
+		)
 		(pin "2"
 		)
@@
 			)
 		)
+		(property "Manufacturer_Part_Number" "MF-PSMF050X-2"
+			(at 172.72 30.48 0)
+			(hide yes)
+			(show_name no)
+			(do_not_autoplace no)
+			(effects
+				(font
+					(size 1.27 1.27)
+				)
+			)
+		)
 		(pin "1"
 		)
@@
 			)
 		)
+		(property "Manufacturer_Part_Number" "MF-PSMF050X-2"
+			(at 158.75 114.3 90)
+			(hide yes)
+			(show_name no)
+			(do_not_autoplace no)
+			(effects
+				(font
+					(size 1.27 1.27)
+				)
+			)
+		)
 		(pin "1"
 		)
@@
 			)
 		)
+		(property "Manufacturer_Part_Number" "SRV05-4"
+			(at 133.35 85.09 0)
+			(hide yes)
+			(show_name no)
+			(do_not_autoplace no)
+			(effects
+				(font
+					(size 1.27 1.27)
+				)
+			)
+		)
 		(pin "6"
 		)
@@
 			)
 		)
+		(property "Manufacturer_Part_Number" "CQ02WGF4701TCE"
+			(at 88.9 49.53 0)
+			(hide yes)
+			(show_name no)
+			(do_not_autoplace no)
+			(effects
+				(font
+					(size 1.27 1.27)
+				)
+			)
+		)
 		(pin "2"
 		)
@@
 		)
 		(property "Description" "Resettable fuse, polymeric positive temperature coefficient"
+			(at 133.35 39.37 0)
+			(hide yes)
+			(show_name no)
+			(do_not_autoplace no)
+			(effects
+				(font
+					(size 1.27 1.27)
+				)
+			)
+		)
+		(property "Manufacturer_Part_Number" "MF-PSMF050X-2"
 			(at 133.35 39.37 0)
 			(hide yes)
@@
 			)
 		)
+		(property "Manufacturer_Part_Number" "TS5A3159ADBVR"
+			(at 168.91 123.19 90)
+			(hide yes)
+			(show_name no)
+			(do_not_autoplace no)
+			(effects
+				(font
+					(size 1.27 1.27)
+				)
+			)
+		)
 		(pin "5"
 		)
@@
 			)
 		)
+		(property "Manufacturer_Part_Number" "SRV05-4"
+			(at 184.15 85.09 0)
+			(hide yes)
+			(show_name no)
+			(do_not_autoplace no)
+			(effects
+				(font
+					(size 1.27 1.27)
+				)
+			)
+		)
 		(pin "6"
 		)
@@
 			)
 		)
+		(property "Manufacturer_Part_Number" "SRV05-4"
+			(at 147.32 168.91 0)
+			(hide yes)
+			(show_name no)
+			(do_not_autoplace no)
+			(effects
+				(font
+					(size 1.27 1.27)
+				)
+			)
+		)
 		(pin "6"
 		)
@@
 			(hide yes)
 			(show_name no)
+			(do_not_autoplace no)
+			(effects
+				(font
+					(size 1.27 1.27)
+				)
+			)
+		)
+		(property "Manufacturer_Part_Number" "MF-PSMF050X-2"
+			(at 179.07 114.3 90)
+			(hide yes)
+			(show_name no)
