File: PCB_Hardware/Boards/BLDC/BLDC_V1.0/Motor_Driver.kicad_sch (KiCad schematic)
At the start: 36 parts, among them Q3 TPH3R70APL, Q4 TPH3R70APL, Q5 TPH3R70APL, Q6 TPH3R70APL, Q7 TPH3R70APL, Q8 TPH3R70APL, U1 DRV8353SRTAR

Commit message: minor BLDC changes and production files for ordering
Parts:
- C15: Manufacturer_Part_Number (none) -> CC0603ZRY5V6BB105; Price (none) -> 0.0065
- C16: Manufacturer_Part_Number (none) -> CL21B473KCFNNNE; Price (none) -> 0.0192
- C17: Manufacturer_Part_Number (none) -> GRM155R62A104KE14D; Price (none) -> 0.013
- C18, C19, C20: Manufacturer_Part_Number (none) -> CL05A105MQ5NNNC
- C21: Manufacturer_Part_Number (none) -> CC0402ZRY5V6BB104; Price (none) -> 0.0015
- C22, C25, C26: Manufacturer_Part_Number (none) -> GRM21BD72A225ME01L
- C28: Manufacturer_Part_Number (none) -> C0805C104K1RACAUTO
- Q3, Q4, Q5, Q6, Q7, Q8: Manufacturer_Part_Number (none) -> TPH3R70APL
- R12, R13, R14: Manufacturer_Part_Number (none) -> LR122WF100NT4E
- R15, R16: Manufacturer_Part_Number (none) -> CQ02WGJ0102TCE
- R32, R37, R38: Manufacturer_Part_Number (none) -> RC0402JR-130RL
- U1: Manufacturer_Part_Number (none) -> DRV8353SRTAR
