File: PCB_Hardware/Boards/BLDC/BLDC_V1.0/USBC.kicad_sch (KiCad schematic)
At the start: 7 parts, among them J11 GT-USB-7010ASV, U10 TPD2E2U06DCK

Commit message: minor BLDC changes and production files for ordering
Parts:
- C37: Manufacturer_Part_Number (none) -> CL10A475MQ8NNNC
- C38: Manufacturer_Part_Number (none) -> CC0402ZRY5V6BB104; Price (none) -> 0.0015
- J11: Manufacturer_Part_Number (none) -> GT-USB-7010ASV
- R47, R48: Manufacturer_Part_Number (none) -> RC0402JR-075K1L
- U10: Manufacturer_Part_Number (none) -> TPD2E2U06DCK
Changed lines of the file:
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@@
+			)
+		)
+		(property "Manufacturer_Part_Number" "CL10A475MQ8NNNC"
+			(at 152.4 69.85 0)
+			(hide yes)
+			(show_name no)
+			(do_not_autoplace no)
+			(effects
+				(font
+					(size 1.27 1.27)
+				)
 			)
 		)
@@
 			)
 		)
+		(property "Manufacturer_Part_Number" "TPD2E2U06DCK"
+			(at 149.86 111.76 90)
+			(hide yes)
+			(show_name no)
+			(do_not_autoplace no)
+			(effects
+				(font
+					(size 1.27 1.27)
+				)
+			)
+		)
 		(pin "1"
 		)
@@
 			)
 		)
+		(property "Manufacturer_Part_Number" "CC0402ZRY5V6BB104"
+			(at 165.1 69.85 0)
+			(hide yes)
+			(show_name no)
+			(do_not_autoplace no)
+			(effects
+				(font
+					(size 1.27 1.27)
+				)
+			)
+		)
+		(property "Price" "0.0015"
+			(at 165.1 69.85 0)
+			(hide yes)
+			(show_name no)
+			(do_not_autoplace no)
+			(effects
+				(font
+					(size 1.27 1.27)
+				)
+			)
+		)
 		(pin "2"
 		)
@@
 			)
 		)
+		(property "Manufacturer_Part_Number" "RC0402JR-075K1L"
+			(at 135.89 86.36 90)
+			(hide yes)
+			(show_name no)
+			(do_not_autoplace no)
+			(effects
+				(font
+					(size 1.27 1.27)
+				)
+			)
+		)
 		(pin "1"
 		)
@@
 			)
 		)
+		(property "Manufacturer_Part_Number" "RC0402JR-075K1L"
+			(at 146.05 88.9 90)
+			(hide yes)
+			(show_name no)
+			(do_not_autoplace no)
+			(effects
+				(font
+					(size 1.27 1.27)
+				)
+			)
+		)
 		(pin "1"
 		)
@@
 			(at 115.57 96.52 0)
 			(hide yes)
+			(show_name no)
+			(do_not_autoplace no)
+			(effects
+				(font
+					(size 1.27 1.27)
+				)
+			)
+		)
+		(property "Manufacturer_Part_Number" "GT-USB-7010ASV"
+			(at 115.57 96.52 0)
+			(hide yes)
